Commit message: Added Nav2

File: description/lidar.xacro (robot description, xacro)
@@ -2,5 +2,5 @@
 <robot xmlns:xacro="http://www.ros.org/wiki/xacro" >
     <joint name="laser_joint" type="fixed">
-        <parent link="chassis"/>
+        <parent link="base_link"/>
         <child link="laser_frame"/>
         <origin xyz="0.1 0 0.1" rpy="0 0 0"/>
@@ -23,8 +23,8 @@
     </link>
     <gazebo reference="laser_frame">
-        <material>Gazebo/Red</material>
+        <material>Gazebo/Blue</material>
         <sensor name="laser" type="ray">
             <pose> 0 0 0 0 0 0 </pose>
-            <visualize>true</visualize>
+            <visualize>false</visualize>
             <update_rate>10</update_rate>
             <ray>

File: description/robot.urdf.xacro (robot description, xacro)
@@ -1,7 +1,13 @@
 <?xml version="1.0"?>
 <robot xmlns:xacro="http://www.ros.org/wiki/xacro"  name="robot">
-    <xacro:include filename="robot_core.xacro"/>
-    <xacro:include filename="inertial_macros.xacro"/>
-    <xacro:include filename="gazebo_control.xacro"/>
-    <xacro:include filename="lidar.xacro"/>
+    <xacro:arg name="use_ros2_control" default="true"/>
+    <xacro:arg name="sim_mode" default="false"/>
+    <xacro:include filename="robot_core.xacro" />
+    <xacro:include filename="lidar.xacro" />
+    <xacro:if value="$(arg use_ros2_control)">
+        <xacro:include filename="ros2_control.xacro" />
+    </xacro:if>
+    <xacro:unless value="$(arg use_ros2_control)">
+        <xacro:include filename="gazebo_control.xacro" />
+    </xacro:unless>
 </robot>

File: description/robot_core.xacro (robot description, xacro)
@@ -21,4 +21,7 @@
         <color rgba="1 1 1 1"/>
     </material>
+    <material name="red">
+        <color rgba="1 0 0 1"/>
+    </material>
     <material name="blue">
         <color rgba="0.2 0.2 1 1"/>
@@ -26,4 +29,10 @@
     <!-- ここに図形情報 (Information of Shapes) -->
     <link name="base_link"/>
+    <link name="base_footprint"/>
+    <joint name="base_footprint_joint" type="fixed">
+        <parent link="base_link"/>
+        <child link="base_footprint"/>
+        <origin xyz="0 0 0" rpy="0 0 0"/>
+    </joint>
     <!-- ボディ (Body) -->
     <link name="chassis">
@@ -55,8 +64,8 @@
         <collision>
             <geometry>
-                <cylinder radius="${wheel_radius}" length="${wheel_thickness}"/>
+                <sphere radius="${wheel_radius}"/>
             </geometry>
         </collision>
-        <xacro:inertial_cylinder mass="0.1" length="${wheel_thickness}" radius="${wheel_radius}">
+        <xacro:inertial_cylinder mass="${wheel_mass}" length="${wheel_thickness}" radius="${wheel_radius}">
             <origin xyz="0 0 0" rpy="0 0 0"/>
         </xacro:inertial_cylinder>
@@ -72,8 +81,8 @@
         <collision>
             <geometry>
-                <cylinder radius="${wheel_radius}" length="${wheel_thickness}"/>
+                <sphere radius="${wheel_radius}"/>
             </geometry>
         </collision>
-         <xacro:inertial_cylinder mass="0.1" length="${wheel_thickness}" radius="${wheel_radius}">
+        <xacro:inertial_cylinder mass="${wheel_mass}" length="${wheel_thickness}" radius="${wheel_radius}">
             <origin xyz="0 0 0" rpy="0 0 0"/>
         </xacro:inertial_cylinder>
@@ -105,5 +114,5 @@
         <parent link="base_link"/>
         <child link="right_wheel"/>
-        <origin xyz="0 ${wheel_offset_y} 0" rpy="-${pi/2} 0 0"/>
+        <origin xyz="0 ${-wheel_offset_y} 0" rpy="${pi/2} 0 0" />
         <axis xyz="0 0 -1"/>
     </joint>
@@ -111,5 +120,5 @@
         <parent link="base_link"/>
         <child link="left_wheel"/>
-        <origin xyz="0 -${wheel_offset_y} 0" rpy="${pi/2} 0 0"/>
+        <origin xyz="0 ${wheel_offset_y} 0" rpy="-${pi/2} 0 0" />
         <axis xyz="0 0 1"/>
     </joint>

Commit message: Fixed Bugs

File: description/lidar.xacro (robot description, xacro)
@@ -25,5 +25,9 @@
         <material>Gazebo/Blue</material>
         <sensor name="laser" type="ray">
+<<<<<<< HEAD
             <pose> 0 0 0 0 0 0 </pose>
+=======
+            <pose> 0 0 0 0 0 3.1416 </pose>
+>>>>>>> acfb3d4 (Fixed Bugs)
             <visualize>false</visualize>
             <update_rate>10</update_rate>
@@ -50,3 +54,7 @@
         </sensor>
     </gazebo>
+<<<<<<< HEAD
 </robot>
+=======
+</robot>
+>>>>>>> acfb3d4 (Fixed Bugs)

File: description/robot_core.xacro (robot description, xacro)
@@ -3,4 +3,5 @@
    <!-- 部品の寸法 (Size of Parts in meters) -->
     <xacro:include filename="inertial_macros.xacro"/>
+<<<<<<< HEAD
     <xacro:property name="chassis_length" value="0.30"/>
     <xacro:property name="chassis_width" value="0.30"/>
@@ -9,9 +10,23 @@
     <xacro:property name="wheel_radius" value="0.1"/>
     <xacro:property name="wheel_thickness" value="0.05"/>
+=======
+    <xacro:property name="chassis_length" value="0.25"/>
+    <xacro:property name="chassis_width" value="0.204"/>
+    <xacro:property name="chassis_height" value="0.10"/>
+    <xacro:property name="chassis_mass" value="1.5"/>
+    <xacro:property name="wheel_radius" value="0.033"/>
+    <xacro:property name="wheel_thickness" value="0.026"/>
+>>>>>>> acfb3d4 (Fixed Bugs)
     <xacro:property name="wheel_mass" value="0.05"/>
     <xacro:property name="wheel_offset_x" value="0.15"/>
+<<<<<<< HEAD
     <xacro:property name="wheel_offset_y" value="${chassis_width/2 + wheel_thickness/2}"/>
     <xacro:property name="wheel_offset_z" value="0"/>
     <xacro:property name="caster_wheel_radius" value="0.05"/>
+=======
+    <xacro:property name="wheel_offset_y" value="0.105"/>
+    <xacro:property name="wheel_offset_z" value="0"/>
+    <xacro:property name="caster_wheel_radius" value="0.017"/>
+>>>>>>> acfb3d4 (Fixed Bugs)
     <xacro:property name="caster_wheel_mass" value="0.01"/>
     <xacro:property name="caster_wheel_offset_x" value="0.075"/>
@@ -109,10 +124,18 @@
         <parent link="base_link"/>
         <child link="chassis"/>
+<<<<<<< HEAD
         <origin xyz="0 0 0"/>
+=======
+        <origin xyz="0 0 ${(chassis_height/2)+0.03}"/>
+>>>>>>> acfb3d4 (Fixed Bugs)
     </joint>
     <joint name="right_wheel_joint" type="continuous">
         <parent link="base_link"/>
         <child link="right_wheel"/>
+<<<<<<< HEAD
         <origin xyz="0 ${-wheel_offset_y} 0" rpy="${pi/2} 0 0" />
+=======
+        <origin xyz="0 -0.115 ${wheel_radius}" rpy="${pi/2} 0 0" />
+>>>>>>> acfb3d4 (Fixed Bugs)
         <axis xyz="0 0 -1"/>
     </joint>
@@ -120,5 +143,9 @@
         <parent link="base_link"/>
         <child link="left_wheel"/>
+<<<<<<< HEAD
         <origin xyz="0 ${wheel_offset_y} 0" rpy="-${pi/2} 0 0" />
+=======
+        <origin xyz="0 0.115 ${wheel_radius}" rpy="-${pi/2} 0 0" />
+>>>>>>> acfb3d4 (Fixed Bugs)
         <axis xyz="0 0 1"/>
     </joint>
@@ -126,5 +153,9 @@
         <parent link="chassis"/>
         <child link="caster_wheel"/>
+<<<<<<< HEAD
         <origin xyz="${caster_wheel_offset_x} 0 ${caster_wheel_offset_z}"/>
+=======
+        <origin xyz="${caster_wheel_offset_x} 0 ${caster_wheel_radius}"/>
+>>>>>>> acfb3d4 (Fixed Bugs)
     </joint>
     <gazebo reference="chassis">

File: description/ros2_control.xacro (robot description, xacro)
@@ -11,5 +11,9 @@
                 <param name="baud_rate">57600</param>
                 <param name="timeout">1000</param>
+<<<<<<< HEAD
                 <param name="enc_counts_per_rev">3436</param>
+=======
+                <param name="enc_counts_per_rev">1975</param>
+>>>>>>> acfb3d4 (Fixed Bugs)
             </hardware>
             <joint name="left_wheel_joint">
@@ -60,3 +64,7 @@
         </plugin>
     </gazebo>
+<<<<<<< HEAD
 </robot>
+=======
+</robot>
+>>>>>>> acfb3d4 (Fixed Bugs)

Commit message: update animove robot model and launch files

File: description/lidar.xacro (robot description, xacro)
@@ -2,7 +2,7 @@
 <robot xmlns:xacro="http://www.ros.org/wiki/xacro" >
     <joint name="laser_joint" type="fixed">
-        <parent link="base_link"/>
+        <parent link="chassis"/>
         <child link="laser_frame"/>
-        <origin xyz="0.1 0 0.1" rpy="0 0 0"/>
+        <origin xyz="-0.08 0 0.11" rpy="0 0 0"/>
     </joint>
     <link name="laser_frame">
@@ -11,5 +11,5 @@
                 <cylinder radius="0.05" length="0.04"/>
             </geometry>
-            <material name="red"/>
+            <material name="blue"/>
         </visual>
         <collision>
@@ -25,10 +25,6 @@
         <material>Gazebo/Blue</material>
         <sensor name="laser" type="ray">
-<<<<<<< HEAD
             <pose> 0 0 0 0 0 0 </pose>
-=======
-            <pose> 0 0 0 0 0 3.1416 </pose>
->>>>>>> acfb3d4 (Fixed Bugs)
-            <visualize>false</visualize>
+            <visualize>true</visualize>
             <update_rate>10</update_rate>
             <ray>
@@ -54,7 +50,3 @@
         </sensor>
     </gazebo>
-<<<<<<< HEAD
 </robot>
-=======
-</robot>
->>>>>>> acfb3d4 (Fixed Bugs)

File: description/robot.urdf.xacro (robot description, xacro)
@@ -5,4 +5,5 @@
     <xacro:include filename="robot_core.xacro" />
     <xacro:include filename="lidar.xacro" />
+    <xacro:include filename="camera.xacro" />
     <xacro:if value="$(arg use_ros2_control)">
         <xacro:include filename="ros2_control.xacro" />

File: description/robot_core.xacro (robot description, xacro)
@@ -1,36 +1,18 @@
 <?xml version="1.0"?>
 <robot xmlns:xacro="http://www.ros.org/wiki/xacro">
-   <!-- 部品の寸法 (Size of Parts in meters) -->
     <xacro:include filename="inertial_macros.xacro"/>
-<<<<<<< HEAD
-    <xacro:property name="chassis_length" value="0.30"/>
-    <xacro:property name="chassis_width" value="0.30"/>
-    <xacro:property name="chassis_height" value="0.10"/>
-    <xacro:property name="chassis_mass" value="1.0"/>
-    <xacro:property name="wheel_radius" value="0.1"/>
-    <xacro:property name="wheel_thickness" value="0.05"/>
-=======
-    <xacro:property name="chassis_length" value="0.25"/>
-    <xacro:property name="chassis_width" value="0.204"/>
-    <xacro:property name="chassis_height" value="0.10"/>
+    <xacro:property name="chassis_radius" value="0.102"/>
+    <xacro:property name="chassis_height" value="0.18"/>
     <xacro:property name="chassis_mass" value="1.5"/>
     <xacro:property name="wheel_radius" value="0.033"/>
     <xacro:property name="wheel_thickness" value="0.026"/>
->>>>>>> acfb3d4 (Fixed Bugs)
     <xacro:property name="wheel_mass" value="0.05"/>
     <xacro:property name="wheel_offset_x" value="0.15"/>
-<<<<<<< HEAD
-    <xacro:property name="wheel_offset_y" value="${chassis_width/2 + wheel_thickness/2}"/>
-    <xacro:property name="wheel_offset_z" value="0"/>
-    <xacro:property name="caster_wheel_radius" value="0.05"/>
-=======
     <xacro:property name="wheel_offset_y" value="0.105"/>
-    <xacro:property name="wheel_offset_z" value="0"/>
+    <xacro:property name="wheel_offset_z" value="0.0"/>
     <xacro:property name="caster_wheel_radius" value="0.017"/>
->>>>>>> acfb3d4 (Fixed Bugs)
     <xacro:property name="caster_wheel_mass" value="0.01"/>
-    <xacro:property name="caster_wheel_offset_x" value="0.075"/>
-    <xacro:property name="caster_wheel_offset_z" value="${wheel_offset_z - wheel_radius + caster_wheel_radius}"/>
-    <!-- 素材情報 (Material Information)) -->
+    <xacro:property name="caster_wheel_offset_x" value="0.08"/>
+    <xacro:property name="caster_wheel_offset_z" value="${-chassis_height/2 - 0.03 + caster_wheel_radius}"/>
     <material name="white">
         <color rgba="1 1 1 1"/>
@@ -42,5 +24,4 @@
         <color rgba="0.2 0.2 1 1"/>
     </material>
-    <!-- ここに図形情報 (Information of Shapes) -->
     <link name="base_link"/>
     <link name="base_footprint"/>
@@ -50,10 +31,9 @@
         <origin xyz="0 0 0" rpy="0 0 0"/>
     </joint>
-    <!-- ボディ (Body) -->
     <link name="chassis">
         <visual>
             <origin xyz="0 0 0"/>
             <geometry>
-                <box size="${chassis_length} ${chassis_width} ${chassis_height}"/>
+                <cylinder radius="${chassis_radius}" length="${chassis_height}"/>
             </geometry>
             <material name="white"/>
@@ -62,12 +42,11 @@
             <origin xyz="0 0 0"/>
             <geometry>
-                <box size="${chassis_length} ${chassis_width} ${chassis_height}"/>
+                <cylinder radius="${chassis_radius}" length="${chassis_height}"/>
             </geometry>
         </collision>
-        <xacro:inertial_box mass="0.5" x="${chassis_length}" y="${chassis_width}" z="${chassis_height}">
+        <xacro:inertial_cylinder mass="0.5" length="${chassis_height}" radius="${chassis_radius}">
             <origin xyz="0 0 0" rpy="0 0 0"/>
-        </xacro:inertial_box>
+        </xacro:inertial_cylinder>
     </link>
-    <!-- 右車輪 (Right Wheel) -->
     <link name="right_wheel">
         <visual>
@@ -86,5 +65,4 @@
         </xacro:inertial_cylinder>
     </link>
-    <!-- 左車輪 (Left Wheel) -->
     <link name="left_wheel">
         <visual>
@@ -103,5 +81,4 @@
         </xacro:inertial_cylinder>
     </link>
-    <!-- 補助輪 (Caster Wheel) -->
     <link name="caster_wheel">
         <visual>
@@ -120,22 +97,29 @@
         </xacro:inertial_sphere>
     </link>
-    <!-- ここに関節情報 (Information of Joints) -->
+    <link name="back_caster_wheel">
+        <visual>
+            <geometry>
+                <sphere radius="${caster_wheel_radius}"/>
+            </geometry>
+            <material name="white"/>
+        </visual>
+        <collision>
+            <geometry>
+                <sphere radius="${caster_wheel_radius}"/>
+            </geometry>
+        </collision>
+        <xacro:inertial_sphere mass="${caster_wheel_mass}" radius="${caster_wheel_radius}">
+            <origin xyz="0 0 0" rpy="0 0 0"/>
+        </xacro:inertial_sphere>
+    </link>
     <joint name="chassis_joint" type="fixed">
         <parent link="base_link"/>
         <child link="chassis"/>
-<<<<<<< HEAD
-        <origin xyz="0 0 0"/>
-=======
         <origin xyz="0 0 ${(chassis_height/2)+0.03}"/>
->>>>>>> acfb3d4 (Fixed Bugs)
     </joint>
     <joint name="right_wheel_joint" type="continuous">
         <parent link="base_link"/>
         <child link="right_wheel"/>
-<<<<<<< HEAD
-        <origin xyz="0 ${-wheel_offset_y} 0" rpy="${pi/2} 0 0" />
-=======
         <origin xyz="0 -0.115 ${wheel_radius}" rpy="${pi/2} 0 0" />
->>>>>>> acfb3d4 (Fixed Bugs)
         <axis xyz="0 0 -1"/>
     </joint>
@@ -143,9 +127,5 @@
         <parent link="base_link"/>
         <child link="left_wheel"/>
-<<<<<<< HEAD
-        <origin xyz="0 ${wheel_offset_y} 0" rpy="-${pi/2} 0 0" />
-=======
         <origin xyz="0 0.115 ${wheel_radius}" rpy="-${pi/2} 0 0" />
->>>>>>> acfb3d4 (Fixed Bugs)
         <axis xyz="0 0 1"/>
     </joint>
@@ -153,14 +133,15 @@
         <parent link="chassis"/>
         <child link="caster_wheel"/>
-<<<<<<< HEAD
         <origin xyz="${caster_wheel_offset_x} 0 ${caster_wheel_offset_z}"/>
-=======
-        <origin xyz="${caster_wheel_offset_x} 0 ${caster_wheel_radius}"/>
->>>>>>> acfb3d4 (Fixed Bugs)
+    </joint>
+    <joint name="back_caster_wheel_joint" type="fixed">
+        <parent link="chassis"/>
+        <child link="back_caster_wheel"/>
+        <origin xyz="${-caster_wheel_offset_x} 0 ${caster_wheel_offset_z}"/>
     </joint>
     <gazebo reference="chassis">
         <material>Gazebo/White</material>
     </gazebo>
-        <gazebo reference="right_wheel">
+    <gazebo reference="right_wheel">
         <material>Gazebo/Red</material>
     </gazebo>
@@ -173,3 +154,8 @@
         <mu2 value="0.001"/>
     </gazebo>
+    <gazebo reference="back_caster_wheel">
+        <material>Gazebo/White</material>
+        <mu1 value="0.001"/>
+        <mu2 value="0.001"/>
+    </gazebo>
 </robot>

File: description/ros2_control.xacro (robot description, xacro)
@@ -11,9 +11,5 @@
                 <param name="baud_rate">57600</param>
                 <param name="timeout">1000</param>
-<<<<<<< HEAD
-                <param name="enc_counts_per_rev">3436</param>
-=======
                 <param name="enc_counts_per_rev">1975</param>
->>>>>>> acfb3d4 (Fixed Bugs)
             </hardware>
             <joint name="left_wheel_joint">
@@ -60,11 +56,7 @@
     <gazebo>
         <plugin name="gazebo_ros2_control" filename="libgazebo_ros2_control.so">
-            <parameters>$(find s_turtlebot)/config/my_controllers.yaml</parameters>
-            <parameters>$(find s_turtlebot)/config/gaz_ros2_ctl_use_sim.yaml</parameters>
+            <parameters>$(find animove)/config/my_controllers.yaml</parameters>
+            <parameters>$(find animove)/config/gaz_ros2_ctl_use_sim.yaml</parameters>
         </plugin>
     </gazebo>
-<<<<<<< HEAD
 </robot>
-=======
-</robot>
->>>>>>> acfb3d4 (Fixed Bugs)
